File: pcb/pcb/pcb.kicad_sch (KiCad schematic)
At the start: 4 parts, among them J1 Conn_01x28_Socket, J2 Conn_01x28_Socket, J3 Conn_01x03_Socket, J4 Conn_01x04_Socket

Commit message: schematic of pcb
Parts:
- added C1: 500u, symbol Device:C
- added C2, C3, C4: 0.1uF, symbol Device:C
- added D1, D2, D3, D4: WS2812B, LED_SMD:LED_WS2812B_PLCC4_5.0x5.0mm_P3.2mm, symbol LED:WS2812B
- added J5: MAX17048, symbol Connector:Conn_01x06_Socket
- added J6: LSM6DS3TR-C, symbol Connector:Conn_01x09_Socket
- added J7: SSD1306, symbol Connector:Conn_01x04_Socket
- added R1: 330, symbol Device:R_US
Connections:
- net +3V3: now also J5.6 (Pin_6), J6.9 (Pin_9), J7.3 (Pin_3)
- net GND: now also C1.2, C2.2, C3.2, C4.2, D1.3 (VSS), D2.3 (VSS), D3.3 (VSS), D4.3 (VSS), J5.5 (Pin_5), J6.7 (Pin_7), J7.4 (Pin_4)
- net GPIO8: now also R1.1
- new net: D1.2 (DOUT), D2.4 (DIN)
- new net: D1.4 (DIN), R1.2
- new net: D2.2 (DOUT), D3.4 (DIN)
- new net: D3.2 (DOUT), D4.4 (DIN)
- new net +BATT: C1.1, C2.1, C3.1, C4.1, D1.1 (VDD), D2.1 (VDD), D3.1 (VDD), D4.1 (VDD)
- new net PICO_SCL: J5.4 (Pin_4), J6.6 (Pin_6), J7.2 (Pin_2)
- new net PICO_SDA: J5.3 (Pin_3), J6.5 (Pin_5), J7.1 (Pin_1)
Other:
- moved on the sheet: J3, J4
