File: pcb/pcb/pcb.kicad_sch (KiCad schematic)
At the start: 35 parts, among them J1 Conn_01x28_Socket, J2 Conn_01x28_Socket, J3 Conn_01x03_Socket, J4 Conn_01x04_Socket, J5 MAX17048, J6 LSM6DS3TR-C, J7 SSD1306, SW1 SW_SPST, U1 TPS61022

Commit message: (Hopefully) done w/ pcb 😭
Parts:
- C1: value 500u -> 100u
Changed lines of the file:
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@@
 			)
 		)
-		(property "Value" "500u"
+		(property "Value" "100u"
 			(at 166.37 106.6799 0)
 			(effects
