File: pcb/pcb/pcb.kicad_pcb (KiCad board)
At the start: 2 copper layers, 83.5 x 129 mm, 28 parts, among them J1 Conn_01x28_Socket, J2 Conn_01x28_Socket, J3 Conn_01x03_Socket, J4 Conn_01x04_Socket, J5 MAX17048, J6 LSM6DS3TR-C, J7 SSD1306, SW1 SW_SPST, U1 TPS61022

Commit message: tweaked a few issues and created GBR and DRILL files
Routing:
- net GND: track 182.9 -> 185.1 mm
Changed lines of the file:
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@@
 			(outputformat 1)
 			(mirror no)
-			(drillshape 1)
+			(drillshape 0)
 			(scaleselection 1)
-			(outputdirectory "")
+			(outputdirectory "drill/")
 		)
 	)
@@
 	)
 	(segment
+		(start 114.72 137.88)
+		(end 112.38 137.88)
+		(width 0.2)
+		(layer "F.Cu")
+		(net 1)
+	)
+	(segment
 		(start 120.2575 64.2425)
 		(end 120.2575 63.7425)
@@
 	)
 	(segment
-		(start 91.2575 119.2575)
-		(end 92 120)
+		(start 112.38 137.88)
+		(end 111.5 137)
 		(width 0.2)
 		(layer "F.Cu")
@@
 	)
 	(segment
-		(start 124 137.88)
-		(end 124 136.5)
+		(start 91.2575 119.2575)
+		(end 92 120)
 		(width 0.2)
 		(layer "F.Cu")
@@
 	)
 	(via
-		(at 124 136.5)
+		(at 111.5 157.5)
 		(size 0.6)
 		(drill 0.3)
@@
 	)
 	(via
-		(at 111.5 157.5)
+		(at 75.5 89.5)
 		(size 0.6)
 		(drill 0.3)
@@
 	)
 	(via
-		(at 75.5 89.5)
+		(at 111.5 137)
 		(size 0.6)
 		(drill 0.3)
