File: pcb/pcb/pcb.kicad_pcb (KiCad board)
At the start: 2 copper layers, 83.5 x 129 mm, 35 parts, among them J1 Conn_01x28_Socket, J2 Conn_01x28_Socket, J3 Conn_01x03_Socket, J4 Conn_01x04_Socket, J5 MAX17048, J6 LSM6DS3TR-C, J7 SSD1306, SW1 SW_SPST, U1 TPS61022

Commit message: (Hopefully) done w/ pcb 😭
Parts:
- C1: value 500u -> 100u
- moved C1 8.10 mm to (109.1, 67.6)
- moved L1 5.99 mm to (101.0, 53.6)
Routing:
- net +BATT: track 135.6 -> 127.6 mm
- net Net-(U1-SW): track 14.5 -> 6.44 mm
- net -BATT: track 190.7 -> 183.1 mm, vias 7 -> 6
- net +5V: track 232.9 -> 235.1 mm
Other:
- board size 83.5 x 129 mm -> 83.5 x 122 mm
- board text added: "ECE 362 Final Project Sonny Chen & Manav Gagvani"
- board text removed: "Sonny and Manav"
